File: Conductivímetro/PCB/version_02/DAMAVA_02.brd (EAGLE design)
At the start: 100.3 x 80 mm, 46 parts, among them IC2 MAX99ESD, IC4 MAX99ESD, U1 74HC4052DIP

Commit message: actualizacion pcb
Parts:
- removed U1: 74HC4052DIP, SparkFun-AnalogIC:DIL16
- added IC1: MAX454CSD, maxim:SO14
- added JP20, JP21: (no value), pinhead:1X01
- added JP22: (no value), jumper:JP1
- JP2: device pinhead:1X02 -> jumper:JP1
- moved JP2 20.6 mm to (78.0, 25.1), turned to 0 degrees
- moved JP1 14.7 mm to (73.2, 27.9)
- moved JP3 14.7 mm to (69.1, 27.9)
- moved JP4 10.9 mm to (46.2, 23.4)
- moved C6 4.58 mm to (78.0, 7.87)
- moved JP6 4.26 mm to (55.1, 46.7)
- moved JP14 2.54 mm to (46.2, 18.0)
- moved JP15 2.54 mm to (46.2, 15.2)
- moved JP18 2.54 mm to (46.2, 12.7)
- moved JP13 2.54 mm to (46.2, 20.8)
- moved JP19 1.98 mm to (83.3, 48.3)
- moved C4 1.52 mm to (91.7, 15.2)
- moved C5 1.52 mm to (87.6, 12.7)
- moved IC3 1.52 mm to (85.6, 21.6)
- moved R4 1.52 mm to (77.0, 18.5)
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Connections:
- removed net N$12: B1.D4, U1.6
- removed net N$13: JP14.1, U1.12
- removed net N$14: JP15.1, U1.14
- removed net N$16: JP13.1, U1.11
- removed net N$18: JP18.1, U1.15
- removed net N$20: IC4.6, IC4.7, JP5.1, JP6.1, U1.13
- new net A0: B1.D6, IC1.14
- new net A1: B1.D5, IC1.1
- new net E: B1.D4, IC1.2
- new net M1: IC1.11, JP13.1
- new net M2: IC1.10, JP14.1
- new net M3: IC1.5, JP15.1
- new net M4: IC1.4, JP18.1
- new net VSEG: IC1.6, IC4.6, IC4.7, JP5.1, JP6.1
- net GND: now also IC1.13; no longer U1.8
- net N$26: now also JP22.1; no longer IC4.5, JP16.1, JP19.1
- net N$3: now also JP2.2, R3.A; no longer B1.D6, U1.10
- net N$5: now also JP2.1; no longer R3.A
- net N$8: now also IC4.5, JP16.1, JP19.1, JP22.2; no longer B1.D5, U1.9
- net VDD: now also IC1.12, JP21.1; no longer JP2.2, U1.16
- net VEE: now also IC1.3, JP20.1; no longer JP2.1, U1.7
Routing:
- net VSEG: track 0.00 -> 52.6 mm
- net E: track 0.00 -> 44.6 mm
- net N$20: track 44.2 -> 0.00 mm
- net N$12: track 39.9 -> 0.00 mm
- net A1: track 0.00 -> 38.3 mm
- net A0: track 0.00 -> 33.4 mm
- net M4: track 0.00 -> 27.5 mm
- net M3: track 0.00 -> 20.8 mm
- net N$3: track 26.5 -> 6.63 mm
- net N$26: track 36.4 -> 19.7 mm
- net -VCC: track 55.1 -> 39.5 mm
- net VEE: track 23.7 -> 8.84 mm
- net +VCC: track 118.1 -> 103.9 mm
- net N$13: track 11.4 -> 0.00 mm
- net N$16: track 11.1 -> 0.00 mm
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