File: Conductivímetro/PCB/version_02/DAMAVA_02.sch (EAGLE design)
At the start: 46 parts, among them IC2 MAX99ESD, IC4 MAX99ESD, U1 74HC4052DIP

Commit message: actualizacion pcb
Parts:
- removed U1: 74HC4052DIP, SparkFun-AnalogIC:74HC4052DIP
- added IC1: MAX454CSD, maxim:MAX454CSD
- added JP20, JP21: (no value), pinhead:PINHD-1X1
- added JP22: (no value), jumper:JP1E
- JP2: device pinhead:PINHD-1X2 -> jumper:JP1E
Connections:
- removed net N$12: B1.D4, U1.INH
- removed net N$13: JP14.1, U1.X0
- removed net N$14: JP15.1, U1.X1
- removed net N$16: JP13.1, U1.X3
- removed net N$18: JP18.1, U1.X2
- removed net N$20: IC4B.-IN, IC4B.OUT, JP5.1, JP6.1, U1.X
- new net A0: B1.*D6, IC1.OUT
- new net A1: B1.*D5, IC1.A1
- new net E: B1.D4, IC1.A0
- new net M1: IC1.IN3, JP13.1
- new net M2: IC1.IN2, JP14.1
- new net M3: IC1.NC, JP15.1
- new net M4: IC1.V-, JP18.1
- new net VSEG: IC1.NC@1, IC4B.-IN, IC4B.OUT, JP5.1, JP6.1
- net GND: now also IC1.-IN; no longer U1.GND
- net N$26: now also JP22.1; no longer IC4B.+IN, JP16.1, JP19.1
- net N$3: now also JP2.2, R3.A; no longer B1.*D6, U1.A
- net N$5: now also JP2.1; no longer R3.A
- net N$8: now also IC4B.+IN, JP16.1, JP19.1, JP22.2; no longer B1.*D5, U1.B
- net VDD: now also IC1.V+, JP21.1; no longer JP2.2, U1.VCC
- net VEE: now also IC1.GND, JP20.1; no longer JP2.1, U1.VEE
Other:
- moved on the sheet: C4, C5, IC3, JP13, JP14, JP15, JP18, R4, R5
